Commit message: leader and follower added

File: mobile_robot/urdf/robot.urdf.xacro (robot description, xacro)
@@ -5,4 +5,5 @@
   <xacro:property name="length" value="0.5"/>
   <xacro:property name="height" value="0.1"/>
+  <xacro:arg name="robot_color" default="Gazebo/Blue"/> <!-- allow spawning with custom colors (e.g., Gazebo/Green for leader) -->
   <xacro:property name="wheel_radius" value="0.06"/>
   <xacro:property name="wheel_width" value="0.03"/>
@@ -65,6 +66,47 @@
   <xacro:wheel prefix="rear_left" x_reflect="-1" y_reflect="1"/>
   <xacro:wheel prefix="rear_right" x_reflect="-1" y_reflect="-1"/>
+  <!-- Base Link Material -->
   <gazebo reference="base_link">
-    <material>Gazebo/Blue</material>
+    <material>$(arg robot_color)</material>
+  </gazebo>
+  <!-- Add Camera Sensor for Follower Drones -->
+  <link name="camera_link">
+    <visual>
+      <geometry>
+        <box size="0.05 0.05 0.05"/>
+      </geometry>
+      <material name="black"/>
+    </visual>
+  </link>
+  <joint name="camera_joint" type="fixed">
+    <parent link="base_link"/>
+    <child link="camera_link"/>
+    <origin xyz="${length/2 + 0.025} 0 0" rpy="0 0 0"/> <!-- at the exact front center -->
+  </joint>
+  <!-- Camera Plugin -->
+  <gazebo reference="camera_link">
+    <sensor type="camera" name="camera">
+      <update_rate>30.0</update_rate>
+      <camera>
+        <horizontal_fov>1.3962634</horizontal_fov>
+        <image>
+          <width>640</width>
+          <height>480</height>
+          <format>R8G8B8</format>
+        </image>
+        <clip>
+          <near>0.02</near>
+          <far>300</far>
+        </clip>
+      </camera>
+      <plugin name="camera_controller" filename="libgazebo_ros_camera.so">
+        <alwaysOn>true</alwaysOn>
+        <updateRate>30.0</updateRate>
+        <cameraName>camera</cameraName>
+        <imageTopicName>image_raw</imageTopicName>
+        <cameraInfoTopicName>camera_info</cameraInfoTopicName>
+        <frameName>camera_link</frameName>
+      </plugin>
+    </sensor>
   </gazebo>
   <!-- Skid Steer Drive Plugin -->
